Commit message: ROS2_V3_25_02

File: cra_description/urdf/cr10_robot.xacro (robot description, xacro)
@@ -44,4 +44,5 @@
   <link  name="world"/>
 <joint name="world_joint" type="fixed">
+    <origin xyz="0 0 0.03" rpy="0 0 0" />
     <parent link="world" />
     <child  link="dummy_link" />

File: cra_description/urdf/cr12_robot.xacro (robot description, xacro)
@@ -48,4 +48,5 @@
   <link  name="world"/>
 <joint name="world_joint" type="fixed">
+    <origin xyz="0 0 0.03" rpy="0 0 0" />
     <parent link="world" />
     <child  link="dummy_link" />

File: cra_description/urdf/cr16_robot.xacro (robot description, xacro)
@@ -44,4 +44,5 @@
   <link  name="world"/>
 <joint name="world_joint" type="fixed">
+    <origin xyz="0 0 0.03" rpy="0 0 0" />
     <parent link="world" />
     <child  link="dummy_link" />

File: cra_description/urdf/cr3_robot.xacro (robot description, xacro)
@@ -44,4 +44,5 @@
   <link  name="world"/>
 <joint name="world_joint" type="fixed">
+    <origin xyz="0 0 0.03" rpy="0 0 0" />
     <parent link="world" />
     <child  link="dummy_link" />

File: cra_description/urdf/cr5_robot.xacro (robot description, xacro)
@@ -33,4 +33,5 @@
   <link  name="world"/>
 <joint name="world_joint" type="fixed">
+    <origin xyz="0 0 0.03" rpy="0 0 0" />
     <parent link="world" />
     <child  link="dummy_link" />

File: cra_description/urdf/cr7_robot.xacro (robot description, xacro)
@@ -47,4 +47,5 @@
 <link  name="world"/>
 <joint name="world_joint" type="fixed">
+    <origin xyz="0 0 0.03" rpy="0 0 0" />
     <parent link="world" />
     <child  link="dummy_link" />

File: cra_description/urdf/nova2_robot.xacro (robot description, xacro)
@@ -24,5 +24,11 @@
         </collision>
     </link>
-  <joint
+    <link  name="world"/>
+    <joint name="world_joint" type="fixed">
+        <origin xyz="0 0 0.03" rpy="0 0 0" />
+        <parent link="world" />
+        <child  link="dummy_link" />
+    </joint>
+    <joint
     name="dummy_joint"
     type="fixed">

File: cra_description/urdf/nova5_robot.xacro (robot description, xacro)
@@ -43,4 +43,10 @@
     </collision>
   </link>
+  <link  name="world"/>
+  <joint name="world_joint" type="fixed">
+        <origin xyz="0 0 0.03" rpy="0 0 0" />
+        <parent link="world" />
+        <child  link="dummy_link" />
+    </joint>
   <joint
     name="dummy_joint"
