Commit message: fix: Fix Nova2 joint axis inconsistency

File: cra_description/urdf/nova2_robot.xacro (robot description, xacro)
@@ -64,5 +64,5 @@
         <parent link="base_link" />
         <child link="Link1" />
-        <axis xyz="0 0 -1" />
+        <axis xyz="0 0 1" />
         <limit lower="-6.28" upper="6.28" effort="300" velocity="100" />
     </joint>
@@ -151,5 +151,5 @@
         <parent link="Link3" />
         <child link="Link4" />
-        <axis xyz="0 0 -1" />
+        <axis xyz="0 0 1" />
         <limit lower="-6.28" upper="6.28" effort="300" velocity="100" />
     </joint>
@@ -180,5 +180,5 @@
         <parent link="Link4" />
         <child link="Link5" />
-        <axis xyz="0 0 -1" />
+        <axis xyz="0 0 1" />
         <limit lower="-6.28" upper="6.28" effort="300" velocity="100" />
     </joint>
